Commit message: added nav2 ros2 contrl and slam but there is a big conrol gap between gazebo and rviz2

File: description/lidar.xacro (robot description, xacro)
@@ -17,7 +17,7 @@
                 </scan>
                 <range>
-                    <min>0.1</min>
+                    <min>0.3</min>
                     <max>12</max>
-                    <resolution>0.01</resolution>
+                    <!-- <resolution>0.01</resolution> -->
                 </range>
             </ray>

File: description/robot.urdf.xacro (robot description, xacro)
@@ -3,5 +3,6 @@
     <!-- <xacro:include filename="robot_core.xacro"/> -->
     <xacro:include filename="robot_core2.xacro"/>
-    <xacro:include filename="gazebo_control.xacro"/>
+    <!-- <xacro:include filename="gazebo_control.xacro"/> -->
+    <xacro:include filename="ros2_control.xacro"/>
     <xacro:include filename="lidar.xacro"/>
 </robot>

File: description/robot_core2.xacro (robot description, xacro)
@@ -55,11 +55,18 @@
     </collision>
   </link>
-  <gazebo reference="base_link">
+  <joint name="base_footprint_joint" type="fixed">
+        <parent link="base_link"/>
+        <child link="base_footprint"/>
+        <origin xyz="0 0 0" rpy="0 0 0"/>
+    </joint>
+  <link name="base_footprint">
+  </link>
+  <!-- <gazebo reference="base_link">
     <material>Gazebo/White</material>
-    <!-- <mu1>0.9</mu1>
-    <mu2>0.9</mu2> -->
-    <kp>500000.0</kp>
-    <kd>100.0</kd>
-  </gazebo>
+    <mu1>0.9</mu1>
+    <mu2>0.9</mu2>
+    <kp>500000.0</kp>
+    <kd>100.0</kd>
+  </gazebo> -->
   <link
     name="front_right_wheel">
@@ -110,5 +117,4 @@
     <minDepth>0.001</minDepth>
     <maxVel>0.1</maxVel>
-    <!-- <fdir1>1 0 0</fdir1> -->
   </gazebo>
   <joint
@@ -173,5 +179,4 @@
     <minDepth>0.001</minDepth>
     <maxVel>0.1</maxVel>
-    <!-- <fdir1>1 0 0</fdir1> -->
   </gazebo>
   <joint
@@ -228,12 +233,11 @@
     </collision>
   </link>
-      <gazebo reference="bottom_right_wheel">
-    <mu1>1</mu1>
-    <mu2>1</mu2>
-    <kp>500000.0</kp>
-    <kd>100.0</kd>
-    <minDepth>0.001</minDepth>
-    <maxVel>0.1</maxVel>
-    <!-- <fdir1>1 0 0</fdir1> -->
+  <gazebo reference="bottom_right_wheel">
+    <mu1>1</mu1>
+    <mu2>1</mu2>
+    <kp>500000.0</kp>
+    <kd>100.0</kd>
+    <minDepth>0.001</minDepth>
+    <maxVel>0.1</maxVel>
   </gazebo>
   <joint
@@ -290,5 +294,5 @@
     </collision>
   </link>
-    <gazebo reference="bottom_left_wheel">
+  <gazebo reference="bottom_left_wheel">
     <material>Gazebo/White</material>
     <mu1>1</mu1>
@@ -298,5 +302,4 @@
     <minDepth>0.001</minDepth>
     <maxVel>0.1</maxVel>
-    <!-- <fdir1>1 0 0</fdir1> -->
   </gazebo>
   <joint
@@ -361,5 +364,4 @@
     <minDepth>0.001</minDepth>
     <maxVel>0.1</maxVel>
-    <!-- <fdir1>1 0 0</fdir1> -->
   </gazebo>
   <joint
@@ -416,5 +418,5 @@
     </collision>
   </link>
-    <gazebo reference="left_tread">
+  <gazebo reference="left_tread">
     <material>Gazebo/Black</material>
     <mu1>1</mu1>
@@ -424,5 +426,4 @@
     <minDepth>0.001</minDepth>
     <maxVel>0.1</maxVel>
-    <!-- <fdir1>1 0 0</fdir1> -->
   </gazebo>
   <joint
@@ -495,33 +496,3 @@
     <material>Gazebo/Black</material>
   </gazebo>
-    <!-- <xacro:macro name="inertial_cylinder" params="mass length radius *origin">
-        <inertial>
-            <xacro:insert_block name="origin"/>
-            <mass value="${mass}" />
-            <inertia ixx="${(1/12) * mass * (3*radius*radius + length*length)}" ixy="0.0" ixz="0.0"
-                    iyy="${(1/12) * mass * (3*radius*radius + length*length)}" iyz="0.0"
-                    izz="${(1/2) * mass * (radius*radius)}" />
-        </inertial>
-    </xacro:macro>
-   <joint name="laser_joint" type="fixed">
-        <parent link="base_link"/>
-        <child link="laser_frame"/>
-        <origin xyz="0.1 0 0.175" rpy="0 0 0"/>
-    </joint>
-    <link name="laser_frame">
-        <visual>
-            <geometry>
-                <cylinder radius="0.05" length="0.04"/>
-            </geometry>
-            <material name="red"/>
-        </visual>
-        <collision>
-            <geometry>
-                <cylinder radius="0.05" length="0.04"/>
-            </geometry>
-        </collision>
-        <xacro:inertial_cylinder mass="0.1" length="0.04" radius="0.05">
-            <origin xyz="0 0 0" rpy="0 0 0"/>
-        </xacro:inertial_cylinder>
-    </link> -->
 </robot>

Commit message: Finished Simulation

File: description/lidar.xacro (robot description, xacro)
@@ -24,5 +24,5 @@
             <plugin name="laser_controller" filename="libgazebo_ros_ray_sensor.so">
                 <ros>
-                    <argument>~/out:=outscan</argument>
+                    <argument>~/out:=scan</argument>
                 </ros>
                 <output_type>sensor_msgs/LaserScan</output_type>

File: description/robot.urdf.xacro (robot description, xacro)
@@ -1,4 +1,4 @@
 <?xml version="1.0"?>
-<robot xmlns:xacro="http://www.ros.org/wiki/xacro" name="rover">
+<robot xmlns:xacro="http://www.ros.org/wiki/xacro" name="robot">
     <!-- <xacro:include filename="robot_core.xacro"/> -->
     <xacro:include filename="robot_core2.xacro"/>

File: description/robot_core.xacro (robot description, xacro)
@@ -26,19 +26,19 @@
       <geometry>
         <mesh
-          filename="file:///home/anonymous/project_ws/src/rover/meshes/base_link.STL" />
-      </geometry>
-      <material
-        name="">
-        <color
-          rgba="0.792156862745098 0.819607843137255 0.933333333333333 1" />
-      </material>
-    </visual>
-    <collision>
-      <origin
-        xyz="0 0 0"
-        rpy="0 0 0" />
-      <geometry>
-        <mesh
-          filename="file:///home/anonymous/project_ws/src/rover/meshes/base_link.STL" />
+          filename="file:///home/anonymous/dev_ws/src/rover/meshes/base_link.STL" />
+      </geometry>
+      <material
+        name="">
+        <color
+          rgba="0.792156862745098 0.819607843137255 0.933333333333333 1" />
+      </material>
+    </visual>
+    <collision>
+      <origin
+        xyz="0 0 0"
+        rpy="0 0 0" />
+      <geometry>
+        <mesh
+          filename="file:///home/anonymous/dev_ws/src/rover/meshes/base_link.STL" />
       </geometry>
     </collision>
@@ -70,19 +70,19 @@
       <geometry>
         <mesh
-          filename="file:///home/anonymous/project_ws/src/rover/meshes/front_right_wheel.STL" />
-      </geometry>
-      <material
-        name="">
-        <color
-          rgba="0.792156862745098 0.819607843137255 0.933333333333333 1" />
-      </material>
-    </visual>
-    <collision>
-      <origin
-        xyz="0 0 0"
-        rpy="0 0 0" />
-      <geometry>
-        <mesh
-          filename="file:///home/anonymous/project_ws/src/rover/meshes/front_right_wheel.STL" />
+          filename="file:///home/anonymous/dev_ws/src/rover/meshes/front_right_wheel.STL" />
+      </geometry>
+      <material
+        name="">
+        <color
+          rgba="0.792156862745098 0.819607843137255 0.933333333333333 1" />
+      </material>
+    </visual>
+    <collision>
+      <origin
+        xyz="0 0 0"
+        rpy="0 0 0" />
+      <geometry>
+        <mesh
+          filename="file:///home/anonymous/dev_ws/src/rover/meshes/front_right_wheel.STL" />
       </geometry>
     </collision>
@@ -123,19 +123,19 @@
       <geometry>
         <mesh
-          filename="file:///home/anonymous/project_ws/src/rover/meshes/front_left_wheel.STL" />
-      </geometry>
-      <material
-        name="">
-        <color
-          rgba="0.792156862745098 0.819607843137255 0.933333333333333 1" />
-      </material>
-    </visual>
-    <collision>
-      <origin
-        xyz="0 0 0"
-        rpy="0 0 0" />
-      <geometry>
-        <mesh
-          filename="file:///home/anonymous/project_ws/src/rover/meshes/front_left_wheel.STL" />
+          filename="file:///home/anonymous/dev_ws/src/rover/meshes/front_left_wheel.STL" />
+      </geometry>
+      <material
+        name="">
+        <color
+          rgba="0.792156862745098 0.819607843137255 0.933333333333333 1" />
+      </material>
+    </visual>
+    <collision>
+      <origin
+        xyz="0 0 0"
+        rpy="0 0 0" />
+      <geometry>
+        <mesh
+          filename="file:///home/anonymous/dev_ws/src/rover/meshes/front_left_wheel.STL" />
       </geometry>
     </collision>
@@ -176,19 +176,19 @@
       <geometry>
         <mesh
-          filename="file:///home/anonymous/project_ws/src/rover/meshes/bottom_right_wheel.STL" />
-      </geometry>
-      <material
-        name="">
-        <color
-          rgba="0.792156862745098 0.819607843137255 0.933333333333333 1" />
-      </material>
-    </visual>
-    <collision>
-      <origin
-        xyz="0 0 0"
-        rpy="0 0 0" />
-      <geometry>
-        <mesh
-          filename="file:///home/anonymous/project_ws/src/rover/meshes/bottom_right_wheel.STL" />
+          filename="file:///home/anonymous/dev_ws/src/rover/meshes/bottom_right_wheel.STL" />
+      </geometry>
+      <material
+        name="">
+        <color
+          rgba="0.792156862745098 0.819607843137255 0.933333333333333 1" />
+      </material>
+    </visual>
+    <collision>
+      <origin
+        xyz="0 0 0"
+        rpy="0 0 0" />
+      <geometry>
+        <mesh
+          filename="file:///home/anonymous/dev_ws/src/rover/meshes/bottom_right_wheel.STL" />
       </geometry>
     </collision>
@@ -229,19 +229,19 @@
       <geometry>
         <mesh
-          filename="file:///home/anonymous/project_ws/src/rover/meshes/bottom_left_wheel.STL" />
-      </geometry>
-      <material
-        name="">
-        <color
-          rgba="0.792156862745098 0.819607843137255 0.933333333333333 1" />
-      </material>
-    </visual>
-    <collision>
-      <origin
-        xyz="0 0 0"
-        rpy="0 0 0" />
-      <geometry>
-        <mesh
-          filename="file:///home/anonymous/project_ws/src/rover/meshes/bottom_left_wheel.STL" />
+          filename="file:///home/anonymous/dev_ws/src/rover/meshes/bottom_left_wheel.STL" />
+      </geometry>
+      <material
+        name="">
+        <color
+          rgba="0.792156862745098 0.819607843137255 0.933333333333333 1" />
+      </material>
+    </visual>
+    <collision>
+      <origin
+        xyz="0 0 0"
+        rpy="0 0 0" />
+      <geometry>
+        <mesh
+          filename="file:///home/anonymous/dev_ws/src/rover/meshes/bottom_left_wheel.STL" />
       </geometry>
     </collision>

File: description/robot_core2.xacro (robot description, xacro)
@@ -37,5 +37,5 @@
       <geometry>
         <mesh
-          filename="file:///home/anonymous/project_ws/src/rover/meshes/base_link.STL" />
+          filename="file:///home/anonymous/dev_ws/src/rover/meshes/base_link.STL" />
       </geometry>
       <material
@@ -51,5 +51,5 @@
       <geometry>
         <mesh
-          filename="file:///home/anonymous/project_ws/src/rover/meshes/base_link.STL" />
+          filename="file:///home/anonymous/dev_ws/src/rover/meshes/base_link.STL" />
       </geometry>
     </collision>
@@ -91,5 +91,5 @@
       <geometry>
         <mesh
-          filename="file:///home/anonymous/project_ws/src/rover/meshes/front_right_wheel.STL" />
+          filename="file:///home/anonymous/dev_ws/src/rover/meshes/front_right_wheel.STL" />
       </geometry>
       <material
@@ -105,5 +105,5 @@
       <geometry>
         <mesh
-          filename="file:///home/anonymous/project_ws/src/rover/meshes/front_right_wheel.STL" />
+          filename="file:///home/anonymous/dev_ws/src/rover/meshes/front_right_wheel.STL" />
       </geometry>
     </collision>
@@ -153,5 +153,5 @@
       <geometry>
         <mesh
-          filename="file:///home/anonymous/project_ws/src/rover/meshes/front_left_wheel.STL" />
+          filename="file:///home/anonymous/dev_ws/src/rover/meshes/front_left_wheel.STL" />
       </geometry>
       <material
@@ -167,5 +167,5 @@
       <geometry>
         <mesh
-          filename="file:///home/anonymous/project_ws/src/rover/meshes/front_left_wheel.STL" />
+          filename="file:///home/anonymous/dev_ws/src/rover/meshes/front_left_wheel.STL" />
       </geometry>
     </collision>
@@ -215,5 +215,5 @@
       <geometry>
         <mesh
-          filename="file:///home/anonymous/project_ws/src/rover/meshes/bottom_right_wheel.STL" />
+          filename="file:///home/anonymous/dev_ws/src/rover/meshes/bottom_right_wheel.STL" />
       </geometry>
       <material
@@ -229,5 +229,5 @@
       <geometry>
         <mesh
-          filename="file:///home/anonymous/project_ws/src/rover/meshes/bottom_right_wheel.STL" />
+          filename="file:///home/anonymous/dev_ws/src/rover/meshes/bottom_right_wheel.STL" />
       </geometry>
     </collision>
@@ -276,5 +276,5 @@
       <geometry>
         <mesh
-          filename="file:///home/anonymous/project_ws/src/rover/meshes/bottom_left_wheel.STL" />
+          filename="file:///home/anonymous/dev_ws/src/rover/meshes/bottom_left_wheel.STL" />
       </geometry>
       <material
@@ -290,5 +290,5 @@
       <geometry>
         <mesh
-          filename="file:///home/anonymous/project_ws/src/rover/meshes/bottom_left_wheel.STL" />
+          filename="file:///home/anonymous/dev_ws/src/rover/meshes/bottom_left_wheel.STL" />
       </geometry>
     </collision>
@@ -338,5 +338,5 @@
       <geometry>
         <mesh
-          filename="file:///home/anonymous/project_ws/src/rover/meshes/right_tread.STL" />
+          filename="file:///home/anonymous/dev_ws/src/rover/meshes/right_tread.STL" />
       </geometry>
       <material
@@ -352,5 +352,5 @@
       <geometry>
         <mesh
-          filename="file:///home/anonymous/project_ws/src/rover/meshes/right_tread.STL" />
+          filename="file:///home/anonymous/dev_ws/src/rover/meshes/right_tread.STL" />
       </geometry>
     </collision>
@@ -400,5 +400,5 @@
       <geometry>
         <mesh
-          filename="file:///home/anonymous/project_ws/src/rover/meshes/left_tread.STL" />
+          filename="file:///home/anonymous/dev_ws/src/rover/meshes/left_tread.STL" />
       </geometry>
       <material
@@ -414,5 +414,5 @@
       <geometry>
         <mesh
-          filename="file:///home/anonymous/project_ws/src/rover/meshes/left_tread.STL" />
+          filename="file:///home/anonymous/dev_ws/src/rover/meshes/left_tread.STL" />
       </geometry>
     </collision>
@@ -462,5 +462,5 @@
       <geometry>
         <mesh
-          filename="file:///home/anonymous/project_ws/src/rover/meshes/lidar_link.STL" />
+          filename="file:///home/anonymous/dev_ws/src/rover/meshes/lidar_link.STL" />
       </geometry>
       <material
@@ -476,5 +476,5 @@
       <geometry>
         <mesh
-          filename="file:///home/anonymous/project_ws/src/rover/meshes/lidar_link.STL" />
+          filename="file:///home/anonymous/dev_ws/src/rover/meshes/lidar_link.STL" />
       </geometry>
     </collision>

File: description/ros2_control.xacro (robot description, xacro)
@@ -1,6 +1,54 @@
 <?xml version="1.0"?>
 <robot xmlns:xacro="http://www.ros.org/wiki/xacro">
-    <!-- <xacro:unless value="$(arg sim_mode)"> -->
-        <ros2_control name="whatever" type="system">
+    <xacro:unless value="$(arg sim_mode)">
+        <ros2_control name="RealRobot" type="system">
+            <hardware>
+                <plugin>diffdrive_arduino/DiffDriveArduino</plugin>
+                <param name="base_link_to_front_right_wheel">base_link_to_front_right_wheel</param>
+                <param name="base_link_to_front_left_wheel">base_link_to_front_left_wheel</param>
+                <param name="base_link_bottom_right_wheel">base_link_bottom_right_wheel</param>
+                <param name="base_link_to_bottom_left_wheel">base_link_to_bottom_left_wheel</param>
+                <param name="loop_rate">1</param>
+                <param name="device">/dev/ttyUSB0</param>
+                <param name="baud_rate">115200</param>
+                <param name="timeout">5000</param>
+                <param name="enc_counts_per_rev">333</param>
+            </hardware>
+            <joint name="base_link_to_front_right_wheel">
+                <command_interface name="velocity">
+                    <param name="min">-10</param>
+                    <param name="max">10</param>
+                </command_interface>
+                <state_interface name="velocity"/>
+                <state_interface name="position"/>
+            </joint>
+            <joint name="base_link_to_front_left_wheel">
+                <command_interface name="velocity">
+                    <param name="min">-10</param>
+                    <param name="max">10</param>
+                </command_interface>
+                <state_interface name="velocity"/>
+                <state_interface name="position"/>
+            </joint>
+            <joint name="base_link_bottom_right_wheel">
+                <command_interface name="velocity">
+                    <param name="min">-10</param>
+                    <param name="max">10</param>
+                </command_interface>
+                <state_interface name="velocity"/>
+                <state_interface name="position"/>
+            </joint>
+            <joint name="base_link_to_bottom_left_wheel">
+                <command_interface name="velocity">
+                    <param name="min">-10</param>
+                    <param name="max">10</param>
+                </command_interface>
+                <state_interface name="velocity"/>
+                <state_interface name="position"/>
+            </joint>
+        </ros2_control>
+    </xacro:unless>
+    <xacro:if value="$(arg sim_mode)">
+        <ros2_control name="GazeboSystem" type="system">
             <hardware>
                 <plugin>gazebo_ros2_control/GazeboSystem</plugin>
@@ -39,7 +87,9 @@
             </joint>
         </ros2_control>
+    </xacro:if>
     <gazebo>
-        <plugin name="gazebo_ros2_control" filename="libgazebo_ros2_control.so"> //plugin that tells gazebo to use the ros2_control
+        <plugin name="gazebo_ros2_control" filename="libgazebo_ros2_control.so">
             <parameters>$(find rover)/config/my_controllers.yaml</parameters>
+            <parameters>$(find rover)/config/gaz_my_controller_use_sim.yaml</parameters>
         </plugin>
     </gazebo>

File: description/testing.xacro (robot description, xacro)
@@ -27,5 +27,5 @@
       <geometry>
         <mesh
-          filename="file:///home/anonymous/project_ws/src/rover/meshes/base_link.STL" />
+          filename="file:///home/anonymous/dev_ws/src/rover/meshes/base_link.STL" />
       </geometry>
       <material
@@ -41,5 +41,5 @@
       <geometry>
         <mesh
-          filename="file:///home/anonymous/project_ws/src/rover/meshes/base_link.STL" />
+          filename="file:///home/anonymous/dev_ws/src/rover/meshes/base_link.STL" />
       </geometry>
     </collision>
@@ -74,5 +74,5 @@
       <geometry>
         <mesh
-          filename="file:///home/anonymous/project_ws/src/rover/meshes/front_right_wheel.STL" />
+          filename="file:///home/anonymous/dev_ws/src/rover/meshes/front_right_wheel.STL" />
       </geometry>
       <material
@@ -88,5 +88,5 @@
       <geometry>
         <mesh
-          filename="file:///home/anonymous/project_ws/src/rover/meshes/front_right_wheel.STL" />
+          filename="file:///home/anonymous/dev_ws/src/rover/meshes/front_right_wheel.STL" />
       </geometry>
     </collision>
@@ -137,5 +137,5 @@
       <geometry>
         <mesh
-          filename="file:///home/anonymous/project_ws/src/rover/meshes/front_left_wheel.STL" />
+          filename="file:///home/anonymous/dev_ws/src/rover/meshes/front_left_wheel.STL" />
       </geometry>
       <material
@@ -151,5 +151,5 @@
       <geometry>
         <mesh
-          filename="file:///home/anonymous/project_ws/src/rover/meshes/front_left_wheel.STL" />
+          filename="file:///home/anonymous/dev_ws/src/rover/meshes/front_left_wheel.STL" />
       </geometry>
     </collision>
@@ -200,5 +200,5 @@
       <geometry>
         <mesh
-          filename="file:///home/anonymous/project_ws/src/rover/meshes/bottom_right_wheel.STL" />
+          filename="file:///home/anonymous/dev_ws/src/rover/meshes/bottom_right_wheel.STL" />
       </geometry>
       <material
@@ -214,5 +214,5 @@
       <geometry>
         <mesh
-          filename="file:///home/anonymous/project_ws/src/rover/meshes/bottom_right_wheel.STL" />
+          filename="file:///home/anonymous/dev_ws/src/rover/meshes/bottom_right_wheel.STL" />
       </geometry>
     </collision>
@@ -262,5 +262,5 @@
       <geometry>
         <mesh
-          filename="file:///home/anonymous/project_ws/src/rover/meshes/bottom_left_wheel.STL" />
+          filename="file:///home/anonymous/dev_ws/src/rover/meshes/bottom_left_wheel.STL" />
       </geometry>
       <material
@@ -276,5 +276,5 @@
       <geometry>
         <mesh
-          filename="file:///home/anonymous/project_ws/src/rover/meshes/bottom_left_wheel.STL" />
+          filename="file:///home/anonymous/dev_ws/src/rover/meshes/bottom_left_wheel.STL" />
       </geometry>
     </collision>
@@ -325,5 +325,5 @@
       <geometry>
         <mesh
-          filename="file:///home/anonymous/project_ws/src/rover/meshes/right_tread.STL" />
+          filename="file:///home/anonymous/dev_ws/src/rover/meshes/right_tread.STL" />
       </geometry>
       <material
@@ -339,5 +339,5 @@
       <geometry>
         <mesh
-          filename="file:///home/anonymous/project_ws/src/rover/meshes/right_tread.STL" />
+          filename="file:///home/anonymous/dev_ws/src/rover/meshes/right_tread.STL" />
       </geometry>
     </collision>
@@ -388,5 +388,5 @@
       <geometry>
         <mesh
-          filename="file:///home/anonymous/project_ws/src/rover/meshes/left_tread.STL" />
+          filename="file:///home/anonymous/dev_ws/src/rover/meshes/left_tread.STL" />
       </geometry>
       <material
@@ -402,5 +402,5 @@
       <geometry>
         <mesh
-          filename="file:///home/anonymous/project_ws/src/rover/meshes/left_tread.STL" />
+          filename="file:///home/anonymous/dev_ws/src/rover/meshes/left_tread.STL" />
       </geometry>
     </collision>
